Commit message: ros20(aruco+opencv)

File: src/move_turtle/urdf/macroed.rudf.xacro (robot description, xacro)
@@ -212,3 +212,27 @@
     <origin xyz="${.707*width+0.04} 0 ${.707*width}"/>
   </joint>
+  <link name="camera_link">
+    <visual>
+      <geometry>
+        <box size="0.01 0.03 0.03"/>
+      </geometry>
+      <material name="black"/>
+    </visual>
+  </link>
+  <joint name="camera_joint" type="fixed">
+    <parent link="box"/>
+    <child link="camera_link"/>
+    <origin xyz = "0 0 0.04" rpy="0 0 0"/>
+  </joint>
+  <gazebo reference="camera_link">
+    <material>
+      Gazebo/Red
+    </material>
+  </gazebo>
+  <joint name="camera_optical_joint" type="fixed">
+    <origin xyz="0 0 0" rpy="${-pi/2} 0 ${-pi/2}"/>
+    <parent link="camera_link"/>
+    <child link="camera_link_optical"/>
+  </joint>
+  <link name="camera_link_optical"/>
 </robot>
