Commit message: ros24(arduino + move_it)

File: src/move_turtle/urdf/turtlebot3_burger.urdf (robot description, URDF)
Before this commit: robot turtlebot3_burger, 9 links, 8 joints
Links:
- added link flag, mass 0.05; collision box size=0.1 0.02 0.02; visual box size=0.1 0.02 0.02
Joints:
- added joint flag_joint: type revolute, parent base_link, child flag, origin xyz=0.025 -0.05 0.14 rpy=0 0 0, axis 0 -1 0, limit lower=0.0 upper=1.57 effort=1000.0 velocity=0.5
- joint camera_joint: origin xyz=0.10 0.0 0.07 rpy=0 0 0 -> xyz=0.05 0.0 0.14 rpy=0 0 0
